File: PCB/RP2040 Devboard.kicad_pcb (KiCad board)
At the start: 4 copper layers, 40 x 100 mm, 98 parts, among them J1 USB_C_Receptacle_USB2.0_14P, J2 USB_C_Receptacle_PowerOnly_6P, J3 Conn_01x10_Pin, J4 Conn_01x10_Pin, J5 Conn_01x03_Pin, Q1 BSS138, SW1 SW_Push, SW10 SW_Push, SW11 SW_Push, SW12 SW_Push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

Commit message: Updated all the files and fixed any caught mistakes
Parts:
- moved C21 24.2 mm to (179.1, 54.4)
- moved U2 0.20 mm to (178.0, 59.2)
- moved C14 0.17 mm to (174.0, 63.6)
- moved R12 0.16 mm to (177.5, 63.6)
Routing:
- net VBUS: track 256.6 -> 256.1 mm, vias 11 -> 9
- net GND: track 87.7 -> 87.6 mm, vias 101 -> 102
Other:
- board text added: "HDC1080 Addr: 1000000 OLED Addr: 0111100 or 0111101 Buzzer: GPIO24 LED: GPIO25 NeoPixels: GPIO14"
- board text removed: "HDC1080 Addr: 1000000 OLED Addr: 0111100 or 0111101 Buzzer: GPIO 24 LED: GPIO25 NeoPixels: GPIO 13"
